File: pcb/tomu.sch (KiCad schematic (older format))
At the start: 21 parts, among them P1 USART0, P2 DEBUG, P3 USB-PCB, P4 RESET_PAD, P5 5V_PAD, P6 3V_PAD, U1 EFM32HG309

Commit message: pcb: update to kicad 5.0
Signed-off-by: Sean Cross <sean@xobs.io>
Parts:
- added XX2: ESD Bag Sticker, symbol usb-pcb:Note
- C1, C2, C3: symbol C_Small -> Device:C_Small; MPN (none) -> ANY; Manufacturer (none) -> ANY
- D1, D2: symbol LED-RESCUE-tomu -> tomu-rescue:LED-RESCUE-tomu; MPN (none) -> ANY; Manufacturer (none) -> ANY
- P1, P2: symbol Conn_01x03 -> tomu-rescue:Conn_01x03
- P3: symbol USB-PCB -> usb-pcb:USB-PCB
- P4, P5, P6: symbol Conn_01x01 -> tomu-rescue:Conn_01x01
- R1, R2, R3, R4: symbol R_Small -> Device:R_Small; MPN (none) -> ANY; Manufacturer (none) -> ANY
- U1: symbol EFM32HG309 -> efm32hg309:EFM32HG309; MPN (none) -> EFM32HG309F64G-B-QFN24; Manufacturer (none) -> ANY
- W1, W2: symbol TEST-RESCUE-tomu -> tomu-rescue:TEST-RESCUE-tomu
- XX1, XX3, XX4: symbol Note -> usb-pcb:Note
Changed lines of the file:
@@
-EESchema Schematic File Version 2
-LIBS:power
-LIBS:device
-LIBS:transistors
-LIBS:conn
-LIBS:linear
-LIBS:regul
-LIBS:74xx
-LIBS:cmos4000
-LIBS:adc-dac
-LIBS:memory
-LIBS:xilinx
-LIBS:microcontrollers
-LIBS:dsp
-LIBS:microchip
-LIBS:analog_switches
-LIBS:motorola
-LIBS:texas
-LIBS:intel
-LIBS:audio
-LIBS:interface
-LIBS:digital-audio
-LIBS:philips
-LIBS:display
-LIBS:cypress
-LIBS:siliconi
-LIBS:opto
-LIBS:atmel
-LIBS:contrib
-LIBS:valves
-LIBS:efm32hg309
-LIBS:usb-pcb
+EESchema Schematic File Version 4
 LIBS:tomu-cache
-EELAYER 25 0
+EELAYER 26 0
 EELAYER END
 $Descr A4 11693 8268
@@
 $EndDescr
 $Comp
-L C_Small C2
+L Device:C_Small C2
 U 1 1 5798B89B
 P 6100 3950
@@
 F 2 "Capacitors_SMD:C_0402" H 6100 3950 50  0001 C CNN
 F 3 "" H 6100 3950 50  0000 C CNN
+F 4 "ANY" H 6100 3950 50  0001 C CNN "MPN"
+F 5 "ANY" H 6100 3950 50  0001 C CNN "Manufacturer"
 	1    6100 3950
 	1    0    0    -1
 $EndComp
 $Comp
-L GND #PWR7
+L power:GND #PWR07
 U 1 1 5798BA02
 P 6200 4250
-F 0 "#PWR7" H 6200 4000 50  0001 C CNN
+F 0 "#PWR07" H 6200 4000 50  0001 C CNN
 F 1 "GND" H 6200 4100 50  0000 C CNN
 F 2 "" H 6200 4250 50  0000 C CNN
@@
 $EndComp
 $Comp
-L C_Small C3
+L Device:C_Small C3
 U 1 1 5798BA32
 P 7000 3850
@@
 F 2 "Capacitors_SMD:C_0402" H 7000 3850 50  0001 C CNN
 F 3 "" H 7000 3850 50  0000 C CNN
+F 4 "ANY" H 7000 3850 50  0001 C CNN "Manufacturer"
+F 5 "ANY" H 7000 3850 50  0001 C CNN "MPN"
 	1    7000 3850
 	1    0    0    -1
 $EndComp
 $Comp
-L C_Small C1
+L Device:C_Small C1
 U 1 1 5798BCD7
 P 5725 4025
@@
 F 2 "Capacitors_SMD:C_0402" H 5725 4025 50  0001 C CNN
 F 3 "" H 5725 4025 50  0000 C CNN
+F 4 "ANY" V 5725 4025 50  0001 C CNN "MPN"
+F 5 "ANY" V 5725 4025 50  0001 C CNN "Manufacturer"
 	1    5725 4025
 	0    1    1    0
 $EndComp
 $Comp
-L USB-PCB P3
+L usb-pcb:USB-PCB P3
 U 1 1 5798BECB
 P 6650 3250
@@
 USB_5V
 $Comp
-L R_Small R3
+L Device:R_Small R3
 U 1 1 5798C3BC
 P 5650 3100
@@
 F 2 "Resistors_SMD:R_0402" H 5650 3100 50  0001 C CNN
 F 3 "" H 5650 3100 50  0000 C CNN
+F 4 "ANY" V 5650 3100 50  0001 C CNN "Manufacturer"
+F 5 "ANY" V 5650 3100 50  0001 C CNN "MPN"
 	1    5650 3100
 	0    1    1    0
 $EndComp
 $Comp
-L R_Small R4
+L Device:R_Small R4
 U 1 1 5798C529
 P 5650 3175
@@
 F 2 "Resistors_SMD:R_0402" H 5650 3175 50  0001 C CNN
 F 3 "" H 5650 3175 50  0000 C CNN
+F 4 "ANY" V 5650 3175 50  0001 C CNN "Manufacturer"
+F 5 "ANY" V 5650 3175 50  0001 C CNN "MPN"
 	1    5650 3175
 	0    1    1    0
@@
 DBG_SWDIO
 $Comp
-L GND #PWR2
+L power:GND #PWR02
 U 1 1 5798EEB6
 P 2800 4100
-F 0 "#PWR2" H 2800 3850 50  0001 C CNN
+F 0 "#PWR02" H 2800 3850 50  0001 C CNN
 F 1 "GND" H 2800 3950 50  0000 C CNN
 F 2 "" H 2800 4100 50  0000 C CNN
@@
 $EndComp
 $Comp
-L +3V3 #PWR6
+L power:+3V3 #PWR06
 U 1 1 5798EF1D
 P 6000 3575
-F 0 "#PWR6" H 6000 3425 50  0001 C CNN
+F 0 "#PWR06" H 6000 3425 50  0001 C CNN
 F 1 "+3V3" H 6000 3715 50  0000 C CNN
 F 2 "" H 6000 3575 50  0000 C CNN
@@
 $EndComp
 $Comp
-L LED-RESCUE-tomu D1
+L tomu-rescue:LED-RESCUE-tomu D1
 U 1 1 5798F0D5
 P 3150 2450
@@
 F 2 "LEDs:LED_0402" H 3150 2450 50  0001 C CNN
 F 3 "" H 3150 2450 50  0000 C CNN
+F 4 "ANY" V 3150 2450 50  0001 C CNN "MPN"
+F 5 "ANY" V 3150 2450 50  0001 C CNN "Manufacturer"
 	1    3150 2450
 	0    1    1    0
 $EndComp
 $Comp
-L LED-RESCUE-tomu D2
+L tomu-rescue:LED-RESCUE-tomu D2
 U 1 1 5798F173
 P 3550 2450
@@
 F 2 "LEDs:LED_0402" H 3550 2450 50  0001 C CNN
 F 3 "" H 3550 2450 50  0000 C CNN
+F 4 "ANY" V 3550 2450 50  0001 C CNN "Manufacturer"
+F 5 "ANY" V 3550 2450 50  0001 C CNN "MPN"
 	1    3550 2450
 	0    1    1    0
 $EndComp
 $Comp
-L R_Small R2
+L Device:R_Small R2
 U 1 1 5798F38A
 P 3750 2200
@@
 F 2 "Resistors_SMD:R_0402" H 3750 2200 50  0001 C CNN
 F 3 "" H 3750 2200 50  0000 C CNN
+F 4 "ANY" V 3750 2200 50  0001 C CNN "MPN"
+F 5 "ANY" V 3750 2200 50  0001 C CNN "Manufacturer"
 	1    3750 2200
 	0    -1   -1   0
 $EndComp
 $Comp
-L R_Small R1
+L Device:R_Small R1
 U 1 1 5798F3FD
 P 3750 1900
@@
 F 2 "Resistors_SMD:R_0402" H 3750 1900 50  0001 C CNN
 F 3 "" H 3750 1900 50  0000 C CNN
+F 4 "ANY" V 3750 1900 50  0001 C CNN "MPN"
+F 5 "ANY" V 3750 1900 50  0001 C CNN "Manufacturer"
 	1    3750 1900
 	0    1    1    0
 $EndComp
 $Comp
-L +3V3 #PWR1
+L power:+3V3 #PWR01
 U 1 1 5798FD73
 P 2650 2850
-F 0 "#PWR1" H 2650 2700 50  0001 C CNN
+F 0 "#PWR01" H 2650 2700 50  0001 C CNN
 F 1 "+3V3" H 2650 2990 50  0000 C CNN
 F 2 "" H 2650 2850 50  0000 C CNN
@@
 $EndComp
 $Comp
-L TEST-RESCUE-tomu W1
+L tomu-rescue:TEST-RESCUE-tomu W1
 U 1 1 57990318
 P 3600 3400
@@
 $EndComp
 $Comp
-L TEST-RESCUE-tomu W2
+L tomu-rescue:TEST-RESCUE-tomu W2
 U 1 1 57990582
 P 3600 3600
@@
 CAP1B
 $Comp
-L +3V3 #PWR3
+L power:+3V3 #PWR03
 U 1 1 579B6568
 P 3350 2425
-F 0 "#PWR3" H 3350 2275 50  0001 C CNN
+F 0 "#PWR03" H 3350 2275 50  0001 C CNN
 F 1 "+3V3" H 3350 2565 50  0000 C CNN
 F 2 "" H 3350 2425 50  0000 C CNN
@@
 $EndComp
 $Comp
-L EFM32HG309 U1
+L efm32hg309:EFM32HG309 U1
 U 1 1 5798B6D7
 P 4400 4175
@@
 F 2 "Housings_DFN_QFN:QFN-24-1EP_5x5mm_Pitch0.65mm" H 4400 4175 60  0001 C CNN
 F 3 "https://www.silabs.com/documents/public/data-sheets/EFM32HG309.pdf" H 4400 4175 60  0001 C CNN
+F 4 "EFM32HG309F64G-B-QFN24" H 4400 4175 50  0001 C CNN "MPN"
+F 5 "ANY" H 4400 4175 50  0001 C CNN "Manufacturer"
 	1    4400 4175
 	1    0    0    -1
@@
 NoConn ~ 4200 3275
 $Comp
-L GND #PWR4
+L power:GND #PWR04
 U 1 1 57A1602A
 P 4030 4035
-F 0 "#PWR4" H 4030 3785 50  0001 C CNN
+F 0 "#PWR04" H 4030 3785 50  0001 C CNN
 F 1 "GND" H 4030 3885 50  0000 C CNN
 F 2 "" H 4030 4035 50  0000 C CNN
@@
 $EndComp
 $Comp
-L Conn_01x03 P2
+L tomu-rescue:Conn_01x03 P2
 U 1 1 5A55837D
 P 2450 4000
@@
 $EndComp
 $Comp
-L PWR_FLAG #FLG1
+L power:PWR_FLAG #FLG01
 U 1 1 5A55865E
 P 6600 3950
-F 0 "#FLG1" H 6600 4025 50  0001 C CNN
+F 0 "#FLG01" H 6600 4025 50  0001 C CNN
 F 1 "PWR_FLAG" H 6600 4100 50  0000 C CNN
 F 2 "" H 6600 3950 50  0001 C CNN
@@
 /RESET
 $Comp
-L Conn_01x01 P4
+L tomu-rescue:Conn_01x01 P4
 U 1 1 5A55B1FF
 P 4200 4600
@@
 $EndComp
 $Comp
-L Conn_01x01 P5
+L tomu-rescue:Conn_01x01 P5
 U 1 1 5A55B8D8
 P 7300 3300
@@
 $EndComp
 $Comp
-L Note XX1
+L usb-pcb:Note XX1
 U 1 1 5A5A1619
 P 1650 2700
@@
 $EndComp
 $Comp
-L Note XX3
+L usb-pcb:Note XX3
 U 1 1 5A603240
 P 1650 3600
@@
 $EndComp
 $Comp
-L Note XX4
+L usb-pcb:Note XX4
 U 1 1 5A6032EF
 P 1650 4050
@@
 	5950 4025 5950 4150
 Wire Wire Line
-	5750 3350 5750 3925
+	5750 3350 5750 3625
 Wire Wire Line
 	5550 3100 5500 3100
@@
 	5500 3175 5550 3175
 Wire Wire Line
-	7000 2800 7000 3750
+	7000 2800 7000 3300
 Wire Wire Line
 	5750 3700 5500 3700
@@
 	3150 2250 3150 1900
 Wire Wire Line
-	3150 2650 3550 2650
+	3150 2650 3350 2650
 Wire Wire Line
 	3350 2425 3350 2650
@@
 	5820 3100 5750 3100
 Wire Wire Line
-	6350 2800 6350 3050
+	6350 2800 6350 2900
 Wire Wire Line
 	6350 2800 7000 2800
@@
 Connection ~ 7000 3300
 Wire Wire Line
-	5515 4150 7000 4150
+	5515 4150 5950 4150
 Connection ~ 6200 4150
 Wire Wire Line
@@
 	7000 4150 7000 3950
 Wire Wire Line
-	5500 3350 6100 3350
-Wire Wire Line
-	6100 3350 6100 3850
+	5500 3350 5750 3350
+Wire Wire Line
+	6100 3350 6100 3625
 Wire Wire Line
 	5515 4150 5515 4125
@@
 	4050 3050 2560 3050
 $Comp
-L Conn_01x03 P1
+L tomu-rescue:Conn_01x03 P1
 U 1 1 5A55AC38
 P 2360 3150
@@
 	2650 3250 2560 3250
 $Comp
-L Conn_01x01 P6
+L tomu-rescue:Conn_01x01 P6
 U 1 1 5A7007C6
 P 5500 2100
@@
 $EndComp
 $Comp
-L +3V3 #PWR5
+L power:+3V3 #PWR05
 U 1 1 5A7008F7
 P 5200 1950
-F 0 "#PWR5" H 5200 1800 50  0001 C CNN
+F 0 "#PWR05" H 5200 1800 50  0001 C CNN
 F 1 "+3V3" H 5200 2090 50  0000 C CNN
 F 2 "" H 5200 1950 50  0001 C CNN
@@
 Wire Wire Line
 	5200 2100 5300 2100
+Wire Wire Line
+	5750 3350 6100 3350
+Wire Wire Line
+	5750 3625 5750 3700
+Wire Wire Line
+	5750 3700 5750 3775
+Wire Wire Line
+	5750 3775 5750 3850
+Wire Wire Line
+	5750 3850 5750 3925
+Wire Wire Line
+	5950 4150 6100 4150
+Wire Wire Line
+	6100 3625 6100 3850
+Wire Wire Line
+	6350 4150 6600 4150
+Wire Wire Line
+	3350 2650 3550 2650
+Wire Wire Line
+	7000 3300 7000 3750
+Wire Wire Line
+	6200 4150 6350 4150
+Wire Wire Line
+	6100 4150 6200 4150
+Wire Wire Line
+	6600 4150 7000 4150
+Wire Wire Line
+	6350 2900 6350 3050
+$Comp
+L usb-pcb:Note XX2
+U 1 1 5B715BCF
+P 1650 3150
+F 0 "XX2" H 1650 3150 60  0000 C CNN
+F 1 "ESD Bag Sticker" H 1650 3050 60  0000 C CNN
+F 2 "" H 1650 3150 60  0001 C CNN
+F 3 "" H 1650 3150 60  0001 C CNN
+F 4 "DNP" H 1650 3150 60  0001 C CNN "Notes"
+F 5 "Black-and-white sticker to affix to ESD bag. 30mm x 50mm" H 1650 3150 60  0001 C CNN "Description"
+	1    1650 3150
+	1    0    0    -1
+$EndComp
 $EndSCHEMATC

Commit message: pcb: set manufacturer of the EFM32 to "Silabs"
Signed-off-by: Sean Cross <sean@xobs.io>
Parts:
- U1: Manufacturer ANY -> Silicon Laboratories Inc
Changed lines of the file:
@@
 F 3 "https://www.silabs.com/documents/public/data-sheets/EFM32HG309.pdf" H 4400 4175 60  0001 C CNN
 F 4 "EFM32HG309F64G-B-QFN24" H 4400 4175 50  0001 C CNN "MPN"
-F 5 "ANY" H 4400 4175 50  0001 C CNN "Manufacturer"
+F 5 "Silicon Laboratories Inc" H 4400 4175 50  0001 C CNN "Manufacturer"
 	1    4400 4175
 	1    0    0    -1
